Commit message: update_bezier_curve

File: robot_description/models/iit-coman-lowerbody-only/model.urdf (robot description, URDF)
Before this commit: robot coman, 31 links, 30 joints
Links:
- link LFoot: geometry collision mesh filename=package://iit-coman/meshes/simple/RoundFoot.STL scale=0.03937 -0.03937 0.03937; visual mesh filename=package://iit-coman/meshes/RoundFoot.STL scale=0.03937 -0.03937 0.03937
- link LFootmot: geometry collision mesh filename=package://iit-coman/meshes/simple/Leg4.STL scale=0.03937 -0.03937 0.03937; visual mesh filename=package://iit-coman/meshes/Leg4.STL scale=0.03937 -0.03937 0.03937
- link LHipMot: geometry collision mesh filename=package://iit-coman/meshes/simple/Leg0.STL scale=0.03937 -0.03937 0.03937; visual mesh filename=package://iit-coman/meshes/Leg0.STL scale=0.03937 -0.03937 0.03937
- link LLowLeg: geometry collision mesh filename=package://iit-coman/meshes/simple/Leg3.STL scale=0.03937 -0.03937 0.03937; visual mesh filename=package://iit-coman/meshes/Leg3.STL scale=0.03937 -0.03937 0.03937
- link LThighLowLeg: geometry collision mesh filename=package://iit-coman/meshes/simple/Leg2.STL scale=0.03937 -0.03937 0.03937; visual mesh filename=package://iit-coman/meshes/Leg2.STL scale=0.03937 -0.03937 0.03937
- link LThighUpLeg: geometry collision mesh filename=package://iit-coman/meshes/simple/Leg1.STL scale=0.03937 -0.03937 0.03937; visual mesh filename=package://iit-coman/meshes/Leg1.STL scale=0.03937 -0.03937 0.03937
- link RFoot: geometry collision mesh filename=package://iit-coman/meshes/simple/RoundFoot.STL scale=0.03937 0.03937 0.03937; visual mesh filename=package://iit-coman/meshes/RoundFoot.STL scale=0.03937 0.03937 0.03937
- link RFootmot: geometry collision mesh filename=package://iit-coman/meshes/simple/Leg4.STL scale=0.03937 0.03937 0.03937; visual mesh filename=package://iit-coman/meshes/Leg4.STL scale=0.03937 0.03937 0.03937
- link RHipMot: geometry collision mesh filename=package://iit-coman/meshes/simple/Leg0.STL scale=0.03937 0.03937 0.03937; visual mesh filename=package://iit-coman/meshes/Leg0.STL scale=0.03937 0.03937 0.03937
- link RLowLeg: geometry collision mesh filename=package://iit-coman/meshes/simple/Leg3.STL scale=0.03937 0.03937 0.03937; visual mesh filename=package://iit-coman/meshes/Leg3.STL scale=0.03937 0.03937 0.03937
- link RThighLowLeg: geometry collision mesh filename=package://iit-coman/meshes/simple/Leg2.STL scale=0.03937 0.03937 0.03937; visual mesh filename=package://iit-coman/meshes/Leg2.STL scale=0.03937 0.03937 0.03937
- link RThighUpLeg: geometry collision mesh filename=package://iit-coman/meshes/simple/Leg1.STL scale=0.03937 0.03937 0.03937; visual mesh filename=package://iit-coman/meshes/Leg1.STL scale=0.03937 0.03937 0.03937
- link Waist: geometry collision mesh filename=package://iit-coman/meshes/simple/Waist.STL scale=0.03937 0.03937 0.03937; visual mesh filename=package://iit-coman/meshes/Waist.STL scale=0.03937 0.03937 0.03937

File: robot_description/models/iit-coman-no-forearms/model.urdf (robot description, URDF)
Before this commit: robot coman, 48 links, 47 joints
Links:
- link DWL: geometry collision mesh filename=package://iit-coman-no-forearms/meshes/simple/Torso1.STL scale=0.03937 0.03937 0.03937; visual mesh filename=package://iit-coman-no-forearms/meshes/Torso1.STL scale=0.03937 0.03937 0.03937
- link DWS: geometry collision mesh filename=package://iit-coman-no-forearms/meshes/simple/Torso2.STL scale=0.03937 0.03937 0.03937; visual mesh filename=package://iit-coman-no-forearms/meshes/Torso2.STL scale=0.03937 0.03937 0.03937
- link DWYTorso: geometry collision mesh filename=package://iit-coman-no-forearms/meshes/simple/Torso3.STL scale=0.03937 0.03937 0.03937; visual mesh filename=package://iit-coman-no-forearms/meshes/Torso3.STL scale=0.03937 0.03937 0.03937
- link LElb: geometry collision mesh filename=package://iit-coman-no-forearms/meshes/simple/Elbow.STL scale=1.0 1.0 1.0; visual mesh filename=package://iit-coman-no-forearms/meshes/Elbow.STL scale=1.0 1.0 1.0
- link LFoot: geometry collision mesh filename=package://iit-coman-no-forearms/meshes/simple/RoundFoot.STL scale=0.03937 -0.03937 0.03937; visual mesh filename=package://iit-coman-no-forearms/meshes/RoundFoot.STL scale=0.03937 -0.03937 0.03937
- link LFootmot: geometry collision mesh filename=package://iit-coman-no-forearms/meshes/simple/Leg4.STL scale=0.03937 -0.03937 0.03937; visual mesh filename=package://iit-coman-no-forearms/meshes/Leg4.STL scale=0.03937 -0.03937 0.03937
- link LForearm: geometry collision mesh filename=package://iit-coman-no-forearms/meshes/simple/ForearmOld.STL scale=0.03937 0.03937 0.03937; visual mesh filename=package://iit-coman-no-forearms/meshes/ForearmOld.STL scale=0.03937 0.03937 0.03937
- link LHipMot: geometry collision mesh filename=package://iit-coman-no-forearms/meshes/simple/Leg0.STL scale=0.03937 -0.03937 0.03937; visual mesh filename=package://iit-coman-no-forearms/meshes/Leg0.STL scale=0.03937 -0.03937 0.03937
- link LLowLeg: geometry collision mesh filename=package://iit-coman-no-forearms/meshes/simple/Leg3.STL scale=0.03937 -0.03937 0.03937; visual mesh filename=package://iit-coman-no-forearms/meshes/Leg3.STL scale=0.03937 -0.03937 0.03937
- link LShp: geometry collision mesh filename=package://iit-coman-no-forearms/meshes/simple/Arm0.STL scale=0.03937 -0.03937 0.03937; visual mesh filename=package://iit-coman-no-forearms/meshes/Arm0.STL scale=0.03937 -0.03937 0.03937
- link LShr: geometry collision mesh filename=package://iit-coman-no-forearms/meshes/simple/Arm1.STL scale=0.03937 -0.03937 0.03937; visual mesh filename=package://iit-coman-no-forearms/meshes/Arm1.STL scale=0.03937 -0.03937 0.03937
- link LShy: geometry collision mesh filename=package://iit-coman-no-forearms/meshes/simple/Arm2.STL scale=0.03937 -0.03937 0.03937; visual mesh filename=package://iit-coman-no-forearms/meshes/Arm2.STL scale=0.03937 -0.03937 0.03937
- link LThighLowLeg: geometry collision mesh filename=package://iit-coman-no-forearms/meshes/simple/Leg2.STL scale=0.03937 -0.03937 0.03937; visual mesh filename=package://iit-coman-no-forearms/meshes/Leg2.STL scale=0.03937 -0.03937 0.03937
- link LThighUpLeg: geometry collision mesh filename=package://iit-coman-no-forearms/meshes/simple/Leg1.STL scale=0.03937 -0.03937 0.03937; visual mesh filename=package://iit-coman-no-forearms/meshes/Leg1.STL scale=0.03937 -0.03937 0.03937
- link RElb: geometry collision mesh filename=package://iit-coman-no-forearms/meshes/simple/Elbow.STL scale=1.0 1.0 1.0; visual mesh filename=package://iit-coman-no-forearms/meshes/Elbow.STL scale=1.0 1.0 1.0
- link RFoot: geometry collision mesh filename=package://iit-coman-no-forearms/meshes/simple/RoundFoot.STL scale=0.03937 0.03937 0.03937; visual mesh filename=package://iit-coman-no-forearms/meshes/RoundFoot.STL scale=0.03937 0.03937 0.03937
- link RFootmot: geometry collision mesh filename=package://iit-coman-no-forearms/meshes/simple/Leg4.STL scale=0.03937 0.03937 0.03937; visual mesh filename=package://iit-coman-no-forearms/meshes/Leg4.STL scale=0.03937 0.03937 0.03937
- link RForearm: geometry collision mesh filename=package://iit-coman-no-forearms/meshes/simple/ForearmOld.STL scale=0.03937 0.03937 0.03937; visual mesh filename=package://iit-coman-no-forearms/meshes/ForearmOld.STL scale=0.03937 0.03937 0.03937
- link RHipMot: geometry collision mesh filename=package://iit-coman-no-forearms/meshes/simple/Leg0.STL scale=0.03937 0.03937 0.03937; visual mesh filename=package://iit-coman-no-forearms/meshes/Leg0.STL scale=0.03937 0.03937 0.03937
- link RLowLeg: geometry collision mesh filename=package://iit-coman-no-forearms/meshes/simple/Leg3.STL scale=0.03937 0.03937 0.03937; visual mesh filename=package://iit-coman-no-forearms/meshes/Leg3.STL scale=0.03937 0.03937 0.03937
- link RShp: geometry collision mesh filename=package://iit-coman-no-forearms/meshes/simple/Arm0.STL scale=0.03937 0.03937 0.03937; visual mesh filename=package://iit-coman-no-forearms/meshes/Arm0.STL scale=0.03937 0.03937 0.03937
- link RShr: geometry collision mesh filename=package://iit-coman-no-forearms/meshes/simple/Arm1.STL scale=0.03937 0.03937 0.03937; visual mesh filename=package://iit-coman-no-forearms/meshes/Arm1.STL scale=0.03937 0.03937 0.03937
- link RShy: geometry collision mesh filename=package://iit-coman-no-forearms/meshes/simple/Arm2.STL scale=0.03937 0.03937 0.03937; visual mesh filename=package://iit-coman-no-forearms/meshes/Arm2.STL scale=0.03937 0.03937 0.03937
- link RThighLowLeg: geometry collision mesh filename=package://iit-coman-no-forearms/meshes/simple/Leg2.STL scale=0.03937 0.03937 0.03937; visual mesh filename=package://iit-coman-no-forearms/meshes/Leg2.STL scale=0.03937 0.03937 0.03937
- link RThighUpLeg: geometry collision mesh filename=package://iit-coman-no-forearms/meshes/simple/Leg1.STL scale=0.03937 0.03937 0.03937; visual mesh filename=package://iit-coman-no-forearms/meshes/Leg1.STL scale=0.03937 0.03937 0.03937
- link Waist: geometry collision mesh filename=package://iit-coman-no-forearms/meshes/simple/Waist.STL scale=0.03937 0.03937 0.03937; visual mesh filename=package://iit-coman-no-forearms/meshes/Waist.STL scale=0.03937 0.03937 0.03937

File: robot_description/models/iit-coman-no-forearms/model_jiatao.urdf (robot description, URDF)
Before this commit: robot coman, 47 links, 46 joints
Links:
- link DWL: geometry collision mesh filename=package://iit-coman/meshes/simple/Torso1.STL scale=0.03937 0.03937 0.03937; visual mesh filename=package://iit-coman/meshes/Torso1.STL scale=0.03937 0.03937 0.03937
- link DWS: geometry collision mesh filename=package://iit-coman/meshes/simple/Torso2.STL scale=0.03937 0.03937 0.03937; visual mesh filename=package://iit-coman/meshes/Torso2.STL scale=0.03937 0.03937 0.03937
- link DWYTorso: geometry collision mesh filename=package://iit-coman/meshes/simple/Torso3.STL scale=0.03937 0.03937 0.03937; visual mesh filename=package://iit-coman/meshes/Torso3.STL scale=0.03937 0.03937 0.03937
- link LElb: geometry collision mesh filename=package://iit-coman/meshes/simple/Elbow.STL scale=1.0 1.0 1.0; visual mesh filename=package://iit-coman/meshes/Elbow.STL scale=1.0 1.0 1.0
- link LFoot: geometry collision mesh filename=package://iit-coman/meshes/simple/RoundFoot.STL scale=0.03937 -0.03937 0.03937; visual mesh filename=package://iit-coman/meshes/RoundFoot.STL scale=0.03937 -0.03937 0.03937
- link LFootmot: geometry collision mesh filename=package://iit-coman/meshes/simple/Leg4.STL scale=0.03937 -0.03937 0.03937; visual mesh filename=package://iit-coman/meshes/Leg4.STL scale=0.03937 -0.03937 0.03937
- link LForearm: geometry collision mesh filename=package://iit-coman/meshes/simple/ForearmOld.STL scale=0.03937 0.03937 0.03937; visual mesh filename=package://iit-coman/meshes/ForearmOld.STL scale=0.03937 0.03937 0.03937
- link LHipMot: geometry collision mesh filename=package://iit-coman/meshes/simple/Leg0.STL scale=0.03937 -0.03937 0.03937; visual mesh filename=package://iit-coman/meshes/Leg0.STL scale=0.03937 -0.03937 0.03937
- link LLowLeg: geometry collision mesh filename=package://iit-coman/meshes/simple/Leg3.STL scale=0.03937 -0.03937 0.03937; visual mesh filename=package://iit-coman/meshes/Leg3.STL scale=0.03937 -0.03937 0.03937
- link LShp: geometry collision mesh filename=package://iit-coman/meshes/simple/Arm0.STL scale=0.03937 -0.03937 0.03937; visual mesh filename=package://iit-coman/meshes/Arm0.STL scale=0.03937 -0.03937 0.03937
- link LShr: geometry collision mesh filename=package://iit-coman/meshes/simple/Arm1.STL scale=0.03937 -0.03937 0.03937; visual mesh filename=package://iit-coman/meshes/Arm1.STL scale=0.03937 -0.03937 0.03937
- link LShy: geometry collision mesh filename=package://iit-coman/meshes/simple/Arm2.STL scale=0.03937 -0.03937 0.03937; visual mesh filename=package://iit-coman/meshes/Arm2.STL scale=0.03937 -0.03937 0.03937
- link LThighLowLeg: geometry collision mesh filename=package://iit-coman/meshes/simple/Leg2.STL scale=0.03937 -0.03937 0.03937; visual mesh filename=package://iit-coman/meshes/Leg2.STL scale=0.03937 -0.03937 0.03937
- link LThighUpLeg: geometry collision mesh filename=package://iit-coman/meshes/simple/Leg1.STL scale=0.03937 -0.03937 0.03937; visual mesh filename=package://iit-coman/meshes/Leg1.STL scale=0.03937 -0.03937 0.03937
- link RElb: geometry collision mesh filename=package://iit-coman/meshes/simple/Elbow.STL scale=1.0 1.0 1.0; visual mesh filename=package://iit-coman/meshes/Elbow.STL scale=1.0 1.0 1.0
- link RFoot: geometry collision mesh filename=package://iit-coman/meshes/simple/RoundFoot.STL scale=0.03937 0.03937 0.03937; visual mesh filename=package://iit-coman/meshes/RoundFoot.STL scale=0.03937 0.03937 0.03937
- link RFootmot: geometry collision mesh filename=package://iit-coman/meshes/simple/Leg4.STL scale=0.03937 0.03937 0.03937; visual mesh filename=package://iit-coman/meshes/Leg4.STL scale=0.03937 0.03937 0.03937
- link RForearm: geometry collision mesh filename=package://iit-coman/meshes/simple/ForearmOld.STL scale=0.03937 0.03937 0.03937; visual mesh filename=package://iit-coman/meshes/ForearmOld.STL scale=0.03937 0.03937 0.03937
- link RHipMot: geometry collision mesh filename=package://iit-coman/meshes/simple/Leg0.STL scale=0.03937 0.03937 0.03937; visual mesh filename=package://iit-coman/meshes/Leg0.STL scale=0.03937 0.03937 0.03937
- link RLowLeg: geometry collision mesh filename=package://iit-coman/meshes/simple/Leg3.STL scale=0.03937 0.03937 0.03937; visual mesh filename=package://iit-coman/meshes/Leg3.STL scale=0.03937 0.03937 0.03937
- link RShp: geometry collision mesh filename=package://iit-coman/meshes/simple/Arm0.STL scale=0.03937 0.03937 0.03937; visual mesh filename=package://iit-coman/meshes/Arm0.STL scale=0.03937 0.03937 0.03937
- link RShr: geometry collision mesh filename=package://iit-coman/meshes/simple/Arm1.STL scale=0.03937 0.03937 0.03937; visual mesh filename=package://iit-coman/meshes/Arm1.STL scale=0.03937 0.03937 0.03937
- link RShy: geometry collision mesh filename=package://iit-coman/meshes/simple/Arm2.STL scale=0.03937 0.03937 0.03937; visual mesh filename=package://iit-coman/meshes/Arm2.STL scale=0.03937 0.03937 0.03937
- link RThighLowLeg: geometry collision mesh filename=package://iit-coman/meshes/simple/Leg2.STL scale=0.03937 0.03937 0.03937; visual mesh filename=package://iit-coman/meshes/Leg2.STL scale=0.03937 0.03937 0.03937
- link RThighUpLeg: geometry collision mesh filename=package://iit-coman/meshes/simple/Leg1.STL scale=0.03937 0.03937 0.03937; visual mesh filename=package://iit-coman/meshes/Leg1.STL scale=0.03937 0.03937 0.03937
- link base_link: geometry collision mesh filename=package://iit-coman/meshes/simple/Waist.STL scale=0.03937 0.03937 0.03937; visual mesh filename=package://iit-coman/meshes/Waist.STL scale=0.03937 0.03937 0.03937
